File: 3. PCB/STM32_NRF24L01_Sleep_mode/STM32_NRF24L01_Sleep_mode.kicad_sch (KiCad schematic)
At the start: 73 parts, among them J1 DEBUG, J2 Power Button, J3 Measure current, J4 NRF24L01+PA+LNA, J6 External I2C, P2 USB_C_Plug_USB2.0, Q3 FDN358P, SW1 SW_Push, SW2 SW_Push, SW3 SW_Push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

Commit message: Refactoring code
Other:
- note added: "Переставлено місцями живлення"
Changed lines of the file:
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@@
     (stroke (width 0) (type default))
   )
-  (wire (pts (xy 303.53 113.03) (xy 267.335 113.03))
+  (wire (pts (xy 339.725 113.03) (xy 267.335 113.03))
     (stroke (width 0) (type default))
   )
@@
     (effects (font (size 1.27 1.27)) (justify left bottom))
   )
+  (text "Переставлено місцями живлення" (at 349.25 181.61 0)
+    (effects (font (size 3 3) bold) (justify left bottom))
+  )
   (text "Optional" (at 303.53 80.01 0)
     (effects (font (size 1.27 1.27)) (justify left bottom))
@@
     )
   )
-  (global_label "ACTION" (shape input) (at 303.53 113.03 0) (fields_autoplaced)
-    (effects (font (size 1.016 1.016) (thickness 0.2032) bold) (justify left))
-    (property "Intersheetrefs" "${INTERSHEET_REFS}" (at 311.4709 113.03 0)
-      (effects (font (size 1.27 1.27)) (justify left) hide)
-    )
+  (global_label "ACTION" (shape input) (at 339.725 113.03 0) (fields_autoplaced)
+    (effects (font (size 1.016 1.016) (thickness 0.2032) bold) (justify left))
+    (property "Intersheetrefs" "${INTERSHEET_REFS}" (at 347.6659 113.03 0)
+      (effects (font (size 1.27 1.27)) (justify left) hide)
+    )
